Commit message: fix:joint

File: assets/urdf/assets.urdf (robot description, URDF)
Before this commit: robot assets, 20 links, 19 joints
Joints:
- removed joint right_ankle_3_3_cube_join
- added joint right_ankle_3_3_cube_joint: type revolute, parent right_ankle_3_3_link, child right_ankle_3_3_cube_link, origin xyz=0 0 0 rpy=0 0 0, axis 0 -1 0, limit lower=-3.14 upper=3.14 effort=100 velocity=1
