Commit message: feat(torque): 统一更新关节扭矩限制和奖励惩罚策略
## 🔧 扭矩限制更新

### 1. URDF 文件 (assets/urdf/assets.urdf)
- Hip pitch: 100 Nm → **2.5 Nm** (控制大腿前后摆动，功率较小)
- Hip yaw/roll: 100 Nm → **8 Nm**
- Knee: 100 Nm → **8 Nm**
- Ankle (1-3, cube, axle, foot): 100 Nm → **2.5 Nm** (脚踝关节，精细控制)
- Toe: 100 Nm → **8 Nm**

### 2. MJCF 模块化文件
- `assets/xmls/models/jiyuan/actuators.xml`: 添加 ctrlrange 和 forcerange
- `assets/xmls/models/jiyuan_fit.xml`: 添加 ctrlrange 和 forcerange
- 所有 actuator 均添加详细注释说明扭矩限制策略

## 🎯 奖励函数增强

### 新增归一化扭矩惩罚函数
- `compute_normalized_torque_penalty()`: 根据不同关节的实际扭矩限制进行归一化
  - Hip pitch 关节: 归一化因子 2.5 Nm
  - Hip yaw/roll/knee/toe: 归一化因子 8 Nm
  - Ankle 关节: 归一化因子 2.5 Nm
- 确保所有关节在 [-1, 1] 范围内公平比较

### 新增能量效率奖励
- `compute_energy_efficiency_reward()`: 计算功率惩罚 (扭矩 × 角速度)
- 用于优化能量消耗

### 导出更新
- 在 `src/rl/rewards/__init__.py` 中导出新函数
- 保持向后兼容性，旧的 `compute_torque_penalty` 仍可用

## 📝 技术细节

**扭矩限制设计理由**:
1. **Hip pitch 2.5 Nm**: 主要控制大腿前后摆动，实际功率需求较小
2. **Hip yaw/roll 8 Nm**: 侧向和旋转运动需要更大扭矩维持稳定
3. **Knee 8 Nm**: 支撑和推进动作需要较大扭矩
4. **Ankle 2.5 Nm**: 精细控制平衡，不需要大扭矩
5. **Toe 8 Nm**: 推进动作需要一定扭矩

**归一化惩罚优势**:
- 避免高扭矩限制关节主导惩罚
- 公平评估所有关节的效率
- 更好地引导策略学习

## 🔍 验证
- ✅ actuators.xml: 16 个扭矩限制设置 (8关节 × 2腿)
- ✅ URDF: 13 个 2.5 Nm + 6 个 8 Nm
- ✅ 新函数已导出并可导入

🤖 Generated with [Claude Code](https://claude.com/claude-code)

Co-Authored-By: Claude Sonnet 4.5 <noreply@anthropic.com>

File: assets/urdf/assets.urdf (robot description, URDF)
Before this commit: robot assets, 20 links, 19 joints
Joints:
- joint right_ankle_1_3_cube_joint: limit lower=-3.14 upper=3.14 effort=100 velocity=1 -> lower=-3.14 upper=3.14 effort=2.5 velocity=1
- joint right_ankle_1_3_joint: limit lower=-3.14 upper=3.14 effort=100 velocity=1 -> lower=-3.14 upper=3.14 effort=2.5 velocity=1
- joint right_ankle_1_3_page_joint: limit lower=-3.14 upper=3.14 effort=100 velocity=1 -> lower=-3.14 upper=3.14 effort=2.5 velocity=1
- joint right_ankle_2_3_cube_joint: limit lower=-3.14 upper=3.14 effort=100 velocity=1 -> lower=-3.14 upper=3.14 effort=2.5 velocity=1
- joint right_ankle_2_3_joint: limit lower=-3.14 upper=3.14 effort=100 velocity=1 -> lower=-3.14 upper=3.14 effort=2.5 velocity=1
- joint right_ankle_2_3_page_joint: limit lower=-3.14 upper=3.14 effort=100 velocity=1 -> lower=-3.14 upper=3.14 effort=2.5 velocity=1
- joint right_ankle_3_3_cube_joint: limit lower=-3.14 upper=3.14 effort=100 velocity=1 -> lower=-3.14 upper=3.14 effort=2.5 velocity=1
- joint right_ankle_3_3_joint: limit lower=-3.14 upper=3.14 effort=100 velocity=1 -> lower=-3.14 upper=3.14 effort=2.5 velocity=1
- joint right_ankle_3_3_page_joint: limit lower=-3.14 upper=3.14 effort=100 velocity=1 -> lower=-3.14 upper=3.14 effort=2.5 velocity=1
- joint right_ankle_axle_joint: limit lower=-3.14 upper=3.14 effort=100 velocity=1 -> lower=-3.14 upper=3.14 effort=2.5 velocity=1
- joint right_ankle_cube_joint: limit lower=-3.14 upper=3.14 effort=100 velocity=1 -> lower=-3.14 upper=3.14 effort=2.5 velocity=1
- joint right_foot_joint: limit lower=-3.14 upper=3.14 effort=100 velocity=1 -> lower=-3.14 upper=3.14 effort=2.5 velocity=1
- joint right_hip_cube_joint: limit lower=-3.14 upper=3.14 effort=100 velocity=1 -> lower=-3.14 upper=3.14 effort=8 velocity=1
- joint right_hip_pitch_engine_joint: limit lower=-3.14 upper=3.14 effort=100 velocity=1 -> lower=-3.14 upper=3.14 effort=2.5 velocity=1
- joint right_hip_roll_joint: limit lower=-3.14 upper=3.14 effort=100 velocity=1 -> lower=-3.14 upper=3.14 effort=8 velocity=1
- joint right_hip_yaw_engine_joint: limit lower=-3.14 upper=3.14 effort=100 velocity=1 -> lower=-3.14 upper=3.14 effort=8 velocity=1
- joint right_knee_joint: limit lower=-3.14 upper=3.14 effort=100 velocity=1 -> lower=-3.14 upper=3.14 effort=8 velocity=1
- joint right_thigh_joint: limit lower=-3.14 upper=3.14 effort=100 velocity=1 -> lower=-3.14 upper=3.14 effort=8 velocity=1
- joint right_toe_joint: limit lower=-3.14 upper=3.14 effort=100 velocity=1 -> lower=-3.14 upper=3.14 effort=8 velocity=1
